File: Circuitry/SAG/SAG.kicad_sch (KiCad schematic)
At the start: 0 parts

Commit message: placed some components
Parts:
- added U1: ESP32, Package_DFN_QFN:QFN-48-1EP_6x6mm_P0.4mm_EP4.3x4.3mm, symbol Espressif:ESP32
- added U2: SCD30, SCD30:MODULE_SCD30, symbol SCD30:SCD30
- added U3: SHT85, SHT85:XDCR_SHT85, symbol SHT85:SHT85
- added U4: VEML7700, 4162:MODULE_4162, symbol 4162:4162
Connections:
- new net: U1.3 (VDD3P3), U1.4 (VDD3P3)
- new net +3.3V: U1.1 (VDDA), U1.43 (VDDA), U1.46 (VDDA)
- new net GND: U1.49 (GND)
